File: SubProjects/Kicad/LedStrip/LedStrip.sch (KiCad schematic (older format))
At the start: 29 parts, among them P1 CONN_01X01, P2 CONN_01X01, P3 CONN_01X01, P4 CONN_01X01, P5 CONN_01X01, P6 CONN_01X01, P7 CONN_01X01, P8 CONN_01X01

Commit message: LEdstrip
Parts:
- P1, P2, P3, P4, P5, P6, P7, P8: footprint Pin_Headers:Pin_Header_Straight_1x01 -> Wire_Pads:SolderWirePad_single_0-8mmDrill
Changed lines of the file:
@@
 F 0 "P1" H 1000 1450 50  0000 C CNN
 F 1 "CONN_01X01" V 1100 1350 50  0000 C CNN
-F 2 "Pin_Headers:Pin_Header_Straight_1x01" H 1000 1350 60  0001 C CNN
+F 2 "Wire_Pads:SolderWirePad_single_0-8mmDrill" H 1000 1350 60  0001 C CNN
 F 3 "" H 1000 1350 60  0000 C CNN
 	1    1000 1350
@@
 F 0 "P2" H 1000 2050 50  0000 C CNN
 F 1 "CONN_01X01" V 1100 1950 50  0000 C CNN
-F 2 "Pin_Headers:Pin_Header_Straight_1x01" H 1000 1950 60  0001 C CNN
+F 2 "Wire_Pads:SolderWirePad_single_0-8mmDrill" H 1000 1950 60  0001 C CNN
 F 3 "" H 1000 1950 60  0000 C CNN
 	1    1000 1950
@@
 F 0 "P3" H 1000 2650 50  0000 C CNN
 F 1 "CONN_01X01" V 1100 2550 50  0000 C CNN
-F 2 "Pin_Headers:Pin_Header_Straight_1x01" H 1000 2550 60  0001 C CNN
+F 2 "Wire_Pads:SolderWirePad_single_0-8mmDrill" H 1000 2550 60  0001 C CNN
 F 3 "" H 1000 2550 60  0000 C CNN
 	1    1000 2550
@@
 F 0 "P4" H 1000 3250 50  0000 C CNN
 F 1 "CONN_01X01" V 1100 3150 50  0000 C CNN
-F 2 "Pin_Headers:Pin_Header_Straight_1x01" H 1000 3150 60  0001 C CNN
+F 2 "Wire_Pads:SolderWirePad_single_0-8mmDrill" H 1000 3150 60  0001 C CNN
 F 3 "" H 1000 3150 60  0000 C CNN
 	1    1000 3150
@@
 F 0 "P5" H 1000 3850 50  0000 C CNN
 F 1 "CONN_01X01" V 1100 3750 50  0000 C CNN
-F 2 "Pin_Headers:Pin_Header_Straight_1x01" H 1000 3750 60  0001 C CNN
+F 2 "Wire_Pads:SolderWirePad_single_0-8mmDrill" H 1000 3750 60  0001 C CNN
 F 3 "" H 1000 3750 60  0000 C CNN
 	1    1000 3750
@@
 F 0 "P6" H 1000 4450 50  0000 C CNN
 F 1 "CONN_01X01" V 1100 4350 50  0000 C CNN
-F 2 "Pin_Headers:Pin_Header_Straight_1x01" H 1000 4350 60  0001 C CNN
+F 2 "Wire_Pads:SolderWirePad_single_0-8mmDrill" H 1000 4350 60  0001 C CNN
 F 3 "" H 1000 4350 60  0000 C CNN
 	1    1000 4350
@@
 F 0 "P7" H 1000 5050 50  0000 C CNN
 F 1 "CONN_01X01" V 1100 4950 50  0000 C CNN
-F 2 "Pin_Headers:Pin_Header_Straight_1x01" H 1000 4950 60  0001 C CNN
+F 2 "Wire_Pads:SolderWirePad_single_0-8mmDrill" H 1000 4950 60  0001 C CNN
 F 3 "" H 1000 4950 60  0000 C CNN
 	1    1000 4950
@@
 F 0 "P8" H 1000 5650 50  0000 C CNN
 F 1 "CONN_01X01" V 1100 5550 50  0000 C CNN
-F 2 "Pin_Headers:Pin_Header_Straight_1x01" H 1000 5550 60  0001 C CNN
+F 2 "Wire_Pads:SolderWirePad_single_0-8mmDrill" H 1000 5550 60  0001 C CNN
 F 3 "" H 1000 5550 60  0000 C CNN
 	1    1000 5550
